Commit message: Move camera base a little bit

File: CustomRobots/robot_arms/models/ur3/ur3.urdf.xacro (robot description, xacro)
@@ -25,5 +25,5 @@
     <xacro:property name="parent_base" value="base_link"/>
     <!-- Posición -->
-    <xacro:property name="cam_base_px" value="0.5"/>
+    <xacro:property name="cam_base_px" value="0.6"/>
     <xacro:property name="cam_base_py" value="0.8"/>
     <xacro:property name="cam_base_pz" value="0.5"/>

Commit message: Move camera base a little bit

File: CustomRobots/robot_arms/models/ur3/ur3.urdf.xacro (robot description, xacro)
@@ -25,5 +25,5 @@
     <xacro:property name="parent_base" value="base_link"/>
     <!-- Posición -->
-    <xacro:property name="cam_base_px" value="0.6"/>
+    <xacro:property name="cam_base_px" value="0.4"/>
     <xacro:property name="cam_base_py" value="0.8"/>
     <xacro:property name="cam_base_pz" value="0.5"/>

Commit message: Change robot pose and camera pose

File: CustomRobots/robot_arms/models/ur3/ur3.urdf.xacro (robot description, xacro)
@@ -25,6 +25,6 @@
     <xacro:property name="parent_base" value="base_link"/>
     <!-- Posición -->
-    <xacro:property name="cam_base_px" value="0.4"/>
-    <xacro:property name="cam_base_py" value="0.8"/>
+    <xacro:property name="cam_base_px" value="0.0"/>
+    <xacro:property name="cam_base_py" value="1.4"/>
     <xacro:property name="cam_base_pz" value="0.5"/>
     <!-- Orientación -->

Commit message: change camera pose

File: CustomRobots/robot_arms/models/ur3/ur3.urdf.xacro (robot description, xacro)
@@ -26,5 +26,5 @@
     <!-- Posición -->
     <xacro:property name="cam_base_px" value="0.0"/>
-    <xacro:property name="cam_base_py" value="1.4"/>
+    <xacro:property name="cam_base_py" value="0.3"/>
     <xacro:property name="cam_base_pz" value="0.5"/>
     <!-- Orientación -->

Commit message: change camera pose

File: CustomRobots/robot_arms/models/ur3/ur3.urdf.xacro (robot description, xacro)
@@ -26,5 +26,5 @@
     <!-- Posición -->
     <xacro:property name="cam_base_px" value="0.0"/>
-    <xacro:property name="cam_base_py" value="0.3"/>
+    <xacro:property name="cam_base_py" value="1.3"/>
     <xacro:property name="cam_base_pz" value="0.5"/>
     <!-- Orientación -->

Commit message: Change sausage spawn pose and stop time

File: CustomRobots/robot_arms/models/ur3/ur3.urdf.xacro (robot description, xacro)
@@ -26,5 +26,5 @@
     <!-- Posición -->
     <xacro:property name="cam_base_px" value="0.0"/>
-    <xacro:property name="cam_base_py" value="1.3"/>
+    <xacro:property name="cam_base_py" value="1.2"/>
     <xacro:property name="cam_base_pz" value="0.5"/>
     <!-- Orientación -->
